Commit message: initial commit

File: urdf/R2.xacro (robot description, xacro)
@@ -1,8 +1,8 @@
 <?xml version="1.0" ?>
 <robot name="R2" xmlns:xacro="http://www.ros.org/wiki/xacro">
-<xacro:include filename="$(find ros2_livox_simulation)/urdf/mid360.xacro" />
-<xacro:include filename="$(find r2_description)/urdf/materials.xacro" />
+<!-- <xacro:include filename="$(find ros2_livox_simulation)/urdf/mid360.xacro" /> -->
+<xacro:include filename="$(find rc2026_field)/urdf/materials.xacro" />
 <!-- <xacro:include filename="$(find r2_description)/urdf/R2.trans" /> -->
-<xacro:include filename="$(find r2_description)/urdf/R2.gazebo" />
+<xacro:include filename="$(find rc2026_field)/urdf/R2.gazebo" />
 <link name="base_link">
   <inertial>
@@ -14,5 +14,5 @@
     <origin xyz="0 0 0" rpy="0 0 0"/>
     <geometry>
-      <mesh filename="file://$(find r2_description)/meshes/base_link.stl" scale="0.001 0.001 0.001"/>
+      <mesh filename="file://$(find rc2026_field)/meshes/base_link.stl" scale="0.001 0.001 0.001"/>
     </geometry>
     <material name="silver"/>
@@ -21,5 +21,5 @@
     <origin xyz="0 0 0" rpy="0 0 0"/>
     <geometry>
-      <mesh filename="file://$(find r2_description)/meshes/base_link.stl" scale="0.001 0.001 0.001"/>
+      <mesh filename="file://$(find rc2026_field)/meshes/base_link.stl" scale="0.001 0.001 0.001"/>
     </geometry>
   </collision>
@@ -34,5 +34,5 @@
     <origin xyz="-0.225 0.27 -0.01" rpy="0 0 0"/>
     <geometry>
-      <mesh filename="file://$(find r2_description)/meshes/wheel_1_1.stl" scale="0.001 0.001 0.001"/>
+      <mesh filename="file://$(find rc2026_field)/meshes/wheel_1_1.stl" scale="0.001 0.001 0.001"/>
     </geometry>
     <material name="silver"/>
@@ -54,5 +54,5 @@
     <origin xyz="0.225 0.27 -0.01" rpy="0 0 0"/>
     <geometry>
-      <mesh filename="file://$(find r2_description)/meshes/wheel_2_1.stl" scale="0.001 0.001 0.001"/>
+      <mesh filename="file://$(find rc2026_field)/meshes/wheel_2_1.stl" scale="0.001 0.001 0.001"/>
     </geometry>
     <material name="silver"/>
@@ -74,5 +74,5 @@
     <origin xyz="0.225 -0.27 -0.01" rpy="0 0 0"/>
     <geometry>
-      <mesh filename="file://$(find r2_description)/meshes/wheel_3_1.stl" scale="0.001 0.001 0.001"/>
+      <mesh filename="file://$(find rc2026_field)/meshes/wheel_3_1.stl" scale="0.001 0.001 0.001"/>
     </geometry>
     <material name="silver"/>
@@ -94,5 +94,5 @@
     <origin xyz="-0.225 -0.27 -0.01" rpy="0 0 0"/>
     <geometry>
-      <mesh filename="file://$(find r2_description)/meshes/wheel_4_1.stl" scale="0.001 0.001 0.001"/>
+      <mesh filename="file://$(find rc2026_field)/meshes/wheel_4_1.stl" scale="0.001 0.001 0.001"/>
     </geometry>
     <material name="silver"/>
@@ -114,5 +114,5 @@
     <origin xyz="-0.32015 0.30715 -0.151" rpy="0 0 0"/>
     <geometry>
-      <mesh filename="file://$(find r2_description)/meshes/mid360_1.stl" scale="0.001 0.001 0.001"/>
+      <mesh filename="file://$(find rc2026_field)/meshes/mid360_1.stl" scale="0.001 0.001 0.001"/>
     </geometry>
     <material name="silver"/>
@@ -121,11 +121,11 @@
     <origin xyz="-0.32015 0.30715 -0.151" rpy="0 0 0"/>
     <geometry>
-      <mesh filename="file://$(find r2_description)/meshes/mid360_1.stl" scale="0.001 0.001 0.001"/>
+      <mesh filename="file://$(find rc2026_field)/meshes/mid360_1.stl" scale="0.001 0.001 0.001"/>
     </geometry>
   </collision>
 </link>
-<xacro:mid360 name="livox" parent="mid360_1" topic="/livox/lidar">
+<!-- <xacro:mid360 name="livox" parent="mid360_1" topic="/livox/lidar">
     <origin xyz="0 0 0" rpy="0 0 0"/>
-</xacro:mid360>
+</xacro:mid360> -->
 <link name="camera_link">
   <visual>
@@ -150,5 +150,5 @@
   <parent link="base_link" />
   <child link="camera_link" />
-  <origin xyz="0.5 0 0.50" rpy="0 1.5708 0" />
+  <origin xyz="0.5 0 0.2" rpy="0 0 0" />
 </joint>
 <joint name="spin_1" type="continuous">

Commit message: 修复小问题

File: urdf/R2.xacro (robot description, xacro)
@@ -2,7 +2,7 @@
 <robot name="R2" xmlns:xacro="http://www.ros.org/wiki/xacro">
 <xacro:include filename="$(find ros2_livox_simulation)/urdf/mid360.xacro" />
-<xacro:include filename="$(find r2_description)/urdf/materials.xacro" />
-<!-- <xacro:include filename="$(find r2_description)/urdf/R2.trans" /> -->
-<xacro:include filename="$(find r2_description)/urdf/R2.gazebo" />
+<xacro:include filename="$(find rc2026_field)/urdf/materials.xacro" />
+<!-- <xacro:include filename="$(find rc2026_field)/urdf/R2.trans" /> -->
+<xacro:include filename="$(find rc2026_field)/urdf/R2.gazebo" />
 <link name="base_link">
   <inertial>
@@ -14,5 +14,5 @@
     <origin xyz="0 0 0" rpy="0 0 0"/>
     <geometry>
-      <mesh filename="file://$(find r2_description)/meshes/base_link.stl" scale="0.001 0.001 0.001"/>
+      <mesh filename="file://$(find rc2026_field)/meshes/base_link.stl" scale="0.001 0.001 0.001"/>
     </geometry>
     <material name="silver"/>
@@ -21,5 +21,5 @@
     <origin xyz="0 0 0" rpy="0 0 0"/>
     <geometry>
-      <mesh filename="file://$(find r2_description)/meshes/base_link.stl" scale="0.001 0.001 0.001"/>
+      <mesh filename="file://$(find rc2026_field)/meshes/base_link.stl" scale="0.001 0.001 0.001"/>
     </geometry>
   </collision>
@@ -34,5 +34,5 @@
     <origin xyz="-0.225 0.27 -0.01" rpy="0 0 0"/>
     <geometry>
-      <mesh filename="file://$(find r2_description)/meshes/wheel_1_1.stl" scale="0.001 0.001 0.001"/>
+      <mesh filename="file://$(find rc2026_field)/meshes/wheel_1_1.stl" scale="0.001 0.001 0.001"/>
     </geometry>
     <material name="silver"/>
@@ -54,5 +54,5 @@
     <origin xyz="0.225 0.27 -0.01" rpy="0 0 0"/>
     <geometry>
-      <mesh filename="file://$(find r2_description)/meshes/wheel_2_1.stl" scale="0.001 0.001 0.001"/>
+      <mesh filename="file://$(find rc2026_field)/meshes/wheel_2_1.stl" scale="0.001 0.001 0.001"/>
     </geometry>
     <material name="silver"/>
@@ -74,5 +74,5 @@
     <origin xyz="0.225 -0.27 -0.01" rpy="0 0 0"/>
     <geometry>
-      <mesh filename="file://$(find r2_description)/meshes/wheel_3_1.stl" scale="0.001 0.001 0.001"/>
+      <mesh filename="file://$(find rc2026_field)/meshes/wheel_3_1.stl" scale="0.001 0.001 0.001"/>
     </geometry>
     <material name="silver"/>
@@ -94,5 +94,5 @@
     <origin xyz="-0.225 -0.27 -0.01" rpy="0 0 0"/>
     <geometry>
-      <mesh filename="file://$(find r2_description)/meshes/wheel_4_1.stl" scale="0.001 0.001 0.001"/>
+      <mesh filename="file://$(find rc2026_field)/meshes/wheel_4_1.stl" scale="0.001 0.001 0.001"/>
     </geometry>
     <material name="silver"/>
@@ -114,5 +114,5 @@
     <origin xyz="-0.32015 0.30715 -0.151" rpy="0 0 0"/>
     <geometry>
-      <mesh filename="file://$(find r2_description)/meshes/mid360_1.stl" scale="0.001 0.001 0.001"/>
+      <mesh filename="file://$(find rc2026_field)/meshes/mid360_1.stl" scale="0.001 0.001 0.001"/>
     </geometry>
     <material name="silver"/>
@@ -121,5 +121,5 @@
     <origin xyz="-0.32015 0.30715 -0.151" rpy="0 0 0"/>
     <geometry>
-      <mesh filename="file://$(find r2_description)/meshes/mid360_1.stl" scale="0.001 0.001 0.001"/>
+      <mesh filename="file://$(find rc2026_field)/meshes/mid360_1.stl" scale="0.001 0.001 0.001"/>
     </geometry>
   </collision>

Commit message: 更新模型, 修复已知问题

File: urdf/R2.xacro (robot description, xacro)
@@ -152,31 +152,23 @@
   <origin xyz="0.5 0 0.50" rpy="0 1.5708 0" />
 </joint>
-<joint name="spin_1" type="continuous">
+<joint name="spin_1" type="fixed">
   <origin xyz="0.225 -0.27 0.01" rpy="0 0 0"/>
   <parent link="base_link"/>
   <child link="wheel_1_1"/>
-  <axis xyz="0.0 1.0 0.0"/>
-  <dynamics damping="1.0" friction="1.0"/>
 </joint>
-<joint name="spin_2" type="continuous">
+<joint name="spin_2" type="fixed">
   <origin xyz="-0.225 -0.27 0.01" rpy="0 0 0"/>
   <parent link="base_link"/>
   <child link="wheel_2_1"/>
-  <axis xyz="0.0 1.0 0.0"/>
-  <dynamics damping="1.0" friction="1.0"/>
 </joint>
-<joint name="spin_3" type="continuous">
+<joint name="spin_3" type="fixed">
   <origin xyz="-0.225 0.27 0.01" rpy="0 0 0"/>
   <parent link="base_link"/>
   <child link="wheel_3_1"/>
-  <axis xyz="0.0 1.0 0.0"/>
-  <dynamics damping="1.0" friction="1.0"/>
 </joint>
-<joint name="spin_4" type="continuous">
+<joint name="spin_4" type="fixed">
   <origin xyz="0.225 0.27 0.01" rpy="0 0 0"/>
   <parent link="base_link"/>
   <child link="wheel_4_1"/>
-  <axis xyz="0.0 1.0 0.0"/>
-  <dynamics damping="1.0" friction="1.0"/>
 </joint>
 <joint name="slide_11" type="fixed">
